File: Hardware/WiFiMonitor.sch (KiCad schematic (older format))
At the start: 0 parts

Commit message: Esch-torreta
RTC DS3231 8 PINES Y USB-B CON REGULADOR LM 1117 3.3V
Parts:
- added BT1, BT2: 3.3V, symbol Battery_Cell
- added C1, C2: 10uCP, symbol CP
- added D1: LED_Small, symbol LED_Small
- added IN1, IN2, IN3, IN4: Conn_01x01_Male, symbol Conn_01x01_Male
- added J1: USB_B, symbol USB_B
- added R1, R2, R3, R4: 2KR, symbol R
- added R11, R13: 4.7KR, symbol R
- added R5, R6, R7, R8: 10KR, symbol R
- added R9: 100R, symbol R
- added U1, U2, U3, U4: 4N25, Housings_DIP:DIP-6_W7.62mm, symbol 4N25
- added U5: ESP8266-12E/ESP-12E, XCVR_ESP8266-12E/ESP-12E, symbol ESP8266-12E/ESP-12E
- added U6: LM1117-3.3, symbol LM1117-3.3
- added U7: DS3231MZ+, SOIC8_150MIL, symbol DS3231MZ+
Connections:
- net labels added: +3.3V, GND, SCL, SDA
- wire segments 0 -> 81
- no-connect marks 0 -> 24
