File: Hardware/WiFiMonitor.sch (KiCad schematic (older format))
At the start: 28 parts, among them J1 USB_B, U1 4N25, U2 4N25, U3 4N25, U4 4N25, U5 ESP8266-12E/ESP-12E, U6 LM1117-3.3, U7 DS3231MZ+

Commit message: Charger
Agregue el MCP73831 manager y el conector de la pila, tambien se cambio el ESP por el conector acondicionado para el esp.
Parts:
- removed BT1: 3.3V, symbol Battery_Cell
- removed C1, C2: 10uCP, symbol CP
- removed D1: LED_Small, symbol LED_Small
- removed U5: ESP8266-12E/ESP-12E, XCVR_ESP8266-12E/ESP-12E, symbol ESP8266-12E/ESP-12E
- removed U6: LM1117-3.3, symbol LM1117-3.3
- added C1: 2.2u, symbol C_Small
- added C2: 10u, symbol C_Small
- added C3: 4.7u, symbol C_Small
- added COMUN1, COMUN2: Conn_01x01_Male, PADS:PAD_5x3mm, symbol Conn_01x01_Male
- added D2: LED_Small, symbol LED_Small
- added D3: D_Schottky, symbol D_Schottky
- added J2: ADAP_ESP, symbol Conn_02x06_Odd_Even
- added J3: Conn_01x02, symbol Conn_01x02
- added J?: SWITCH2, symbol Conn_01x02
- added R10, R12, R14, R16: 10K, symbol R
- added R15: 1K, symbol R
- added U5: MCP73831T-4ADI/OT, SOT95P280X145-5N, symbol MCP73831T-4ADI/OT
- added U6: AP1117-33, TO_SOT_Packages_SMD:SOT-223-3Lead_TabPin2, symbol AP1117-33
- BT2: footprint (none) -> Connectors:PINHEAD1-2
- IN1, IN2, IN3, IN4: footprint (none) -> PADS:PAD_5x3mm
- J1: footprint (none) -> Connectors_USB:USB_Micro-B_Wuerth-629105150521
- R1, R11, R13, R3, R4, R5, R6, R7, R8: footprint (none) -> Resistors_SMD:R_0603
- R2: footprint (none) -> Resistors_SMD:R_0603; Fieldname (none) -> Value; manf (none) -> RN731JTTD2101D25
- R9: value 100R -> 10K
- U7: footprint SOIC8_150MIL -> DS3231MZ_:SOIC8_150MIL
Connections:
- net labels added: BAT, CH, D0, D1, D2, D3, GPIO15, GPIO2, RST, VBUS
- wire segments 81 -> 129
- no-connect marks 24 -> 7
Other:
- moved on the sheet: BT2, R11, R13, U7

Commit message: Final
Corregi nombres, y agregue el circuito de programación
Parts:
- removed J1: USB_B, Connectors_USB:USB_Micro-B_Wuerth-629105150521, symbol USB_B
- removed J2: ADAP_ESP, symbol Conn_02x06_Odd_Even
- removed J?: SWITCH2, symbol Conn_01x02
- added BOTTOM_BOOT1, BOTTOM_RST2: KMR221GLFS, SW_KMR221GLFS, symbol KMR221GLFS
- added D1: LED_ON, LEDs:LED_0603, symbol LED_Small
- added D4: RB161, Diodes_SMD:D_SOD-123, symbol D_Schottky
- added J4: ADAP_ESP, Pin_Headers:Pin_Header_Straight_2x08_Pitch2.54mm, symbol Conn_02x08_Top_Bottom
- added J5: FTDI, Pin_Headers:Pin_Header_Straight_1x05_Pitch2.54mm, symbol Conn_01x05
- added R17: 1K, Resistors_SMD:R_0603, symbol R
- added R18: 10K, Resistors_SMD:R_0603, symbol R
- BTRTC1: renamed from BT2; footprint Connectors:PINHEAD1-2 -> Battery_Holders:Keystone_1058_1x2032-CoinCell
- C1, C2, C3: footprint (none) -> Capacitors_SMD:C_0603
- COMUN1: value Conn_01x01_Male -> NC
- COMUN2: value Conn_01x01_Male -> TORRETA
- D2: value LED_Small -> LED_CHAR; footprint (none) -> LEDs:LED_0603
- D3: value D_Schottky -> RB161; footprint (none) -> Diodes_SMD:D_SOD-123
- IN1: value Conn_01x01_Male -> 0_IN
- IN2: value Conn_01x01_Male -> 1_IN
- IN3: value Conn_01x01_Male -> 2_IN
- IN4: value Conn_01x01_Male -> 3_IN
- J3: value Conn_01x02 -> BATT; footprint (none) -> Connectors:PINHEAD1-2
- R1, R2, R3, R4: value 2KR -> 2K
- R10, R12, R14, R15, R16, R9: footprint (none) -> Resistors_SMD:R_0603
- R11, R13: value 4.7KR -> 4.7K
- R5, R6, R7, R8: value 10KR -> 10K
- U5: footprint SOT95P280X145-5N -> MCP73831T-4ADI_OT:SOT95P280X145-5N
Connections:
- net labels added: GNDA, GPIO0, RX, TX, VCC
- net labels removed: VBUS
- wire segments 129 -> 150
- no-connect marks 7 -> 10
Other:
- moved on the sheet: C1, C3, COMUN1, COMUN2, D3, R10, R12, R9, U6

Commit message: PULL_UP_BOTTON
RESISTENCIAS CORREGIDAS PULL UP DEL RTC Y CAMBIO DE BOTON
Parts:
- removed BOTTOM_BOOT1, BOTTOM_RST2: KMR221GLFS, SW_KMR221GLFS, symbol KMR221GLFS
- added S?: BOTTON_BOOT, SW_B3U-1000P, symbol B3U-1000P
- added S?: BOTTON_RST, SW_B3U-1000P, symbol B3U-1000P
Connections:
- wire segments 150 -> 144
Other:
- moved on the sheet: R10, R11, R13
Changed lines of the file:
@@
 LIBS:valves
 LIBS:MCP73831T-4ADI_OT
-LIBS:KMR221GLFS
+LIBS:B3U-1000P
 LIBS:WiFiMonitor-cache
 EELAYER 25 0
@@
 L R R11
 U 1 1 5A4A6EBD
-P 4550 1500
-F 0 "R11" V 4630 1500 50  0000 C CNN
-F 1 "4.7K" V 4550 1500 50  0000 C CNN
-F 2 "Resistors_SMD:R_0603" V 4480 1500 50  0001 C CNN
-F 3 "" H 4550 1500 50  0001 C CNN
-	1    4550 1500
-	0    1    1    0
+P 4450 1300
+F 0 "R11" V 4530 1300 50  0000 C CNN
+F 1 "4.7K" V 4450 1300 50  0000 C CNN
+F 2 "Resistors_SMD:R_0603" V 4380 1300 50  0001 C CNN
+F 3 "" H 4450 1300 50  0001 C CNN
+	1    4450 1300
+	-1   0    0    1
 $EndComp
 $Comp
 L R R13
 U 1 1 5A4A6F12
-P 6650 1300
-F 0 "R13" V 6730 1300 50  0000 C CNN
-F 1 "4.7K" V 6650 1300 50  0000 C CNN
-F 2 "Resistors_SMD:R_0603" V 6580 1300 50  0001 C CNN
-F 3 "" H 6650 1300 50  0001 C CNN
-	1    6650 1300
-	0    1    1    0
+P 6600 1100
+F 0 "R13" V 6680 1100 50  0000 C CNN
+F 1 "4.7K" V 6600 1100 50  0000 C CNN
+F 2 "Resistors_SMD:R_0603" V 6530 1100 50  0001 C CNN
+F 3 "" H 6600 1100 50  0001 C CNN
+	1    6600 1100
+	-1   0    0    1
 $EndComp
 $Comp
@@
 	1    0    0    -1
 $EndComp
-Text Label 4250 1500 0    60   ~ 0
-SCL
-Text Label 6950 1300 0    60   ~ 0
+Text Label 6800 1300 0    60   ~ 0
 SDA
 $Comp
@@
 L +3.3V #PWR018
 U 1 1 5A4E3EAB
-P 4550 5150
-F 0 "#PWR018" H 4550 5000 50  0001 C CNN
-F 1 "+3.3V" H 4550 5290 50  0000 C CNN
-F 2 "" H 4550 5150 50  0001 C CNN
-F 3 "" H 4550 5150 50  0001 C CNN
-	1    4550 5150
+P 4500 5150
+F 0 "#PWR018" H 4500 5000 50  0001 C CNN
+F 1 "+3.3V" H 4500 5290 50  0000 C CNN
+F 2 "" H 4500 5150 50  0001 C CNN
+F 3 "" H 4500 5150 50  0001 C CNN
+	1    4500 5150
 	1    0    0    -1
 $EndComp
@@
 L R R10
 U 1 1 5A4E4153
-P 4550 5800
-F 0 "R10" V 4630 5800 50  0000 C CNN
-F 1 "10K" V 4550 5800 50  0000 C CNN
-F 2 "Resistors_SMD:R_0603" V 4480 5800 50  0001 C CNN
-F 3 "" H 4550 5800 50  0001 C CNN
-	1    4550 5800
+P 4500 5800
+F 0 "R10" V 4580 5800 50  0000 C CNN
+F 1 "10K" V 4500 5800 50  0000 C CNN
+F 2 "Resistors_SMD:R_0603" V 4430 5800 50  0001 C CNN
+F 3 "" H 4500 5800 50  0001 C CNN
+	1    4500 5800
 	1    0    0    -1
 $EndComp
@@
 Text Label 5300 6900 1    60   ~ 0
 CH
-Text Label 4550 6200 1    60   ~ 0
+Text Label 4500 6200 1    60   ~ 0
 RST
 $Comp
 L GND #PWR020
 U 1 1 5A4C5C3E
-P 4550 6950
-F 0 "#PWR020" H 4550 6700 50  0001 C CNN
-F 1 "GND" H 4550 6800 50  0000 C CNN
-F 2 "" H 4550 6950 50  0001 C CNN
-F 3 "" H 4550 6950 50  0001 C CNN
-	1    4550 6950
+P 4500 7450
+F 0 "#PWR020" H 4500 7200 50  0001 C CNN
+F 1 "GND" H 4500 7300 50  0000 C CNN
+F 2 "" H 4500 7450 50  0001 C CNN
+F 3 "" H 4500 7450 50  0001 C CNN
+	1    4500 7450
 	1    0    0    -1
 $EndComp
@@
 L GND #PWR024
 U 1 1 5A4FDC73
-P 3750 6850
-F 0 "#PWR024" H 3750 6600 50  0001 C CNN
-F 1 "GND" H 3750 6700 50  0000 C CNN
-F 2 "" H 3750 6850 50  0001 C CNN
-F 3 "" H 3750 6850 50  0001 C CNN
-	1    3750 6850
+P 3750 7450
+F 0 "#PWR024" H 3750 7200 50  0001 C CNN
+F 1 "GND" H 3750 7300 50  0000 C CNN
+F 2 "" H 3750 7450 50  0001 C CNN
+F 3 "" H 3750 7450 50  0001 C CNN
+	1    3750 7450
 	1    0    0    -1
 $EndComp
@@
 GPIO0
 $Comp
-L KMR221GLFS BOTTOM_BOOT1
-U 1 1 5A4E7485
-P 3750 6300
-F 0 "BOTTOM_BOOT1" H 3650 6390 50  0000 L BNN
-F 1 "KMR221GLFS" H 3640 6050 50  0000 L BNN
-F 2 "SW_KMR221GLFS" H 3750 6300 50  0001 L BNN
-F 3 "401-1427-1-ND" H 3750 6300 50  0001 L BNN
-F 4 "C&K Components" H 3750 6300 50  0001 L BNN "Field4"
-F 5 "None" H 3750 6300 50  0001 L BNN "Field5"
-F 6 "KMR221GLFS" H 3750 6300 50  0001 L BNN "Field6"
-F 7 "https://www.digikey.com.mx/product-detail/en/c-k/KMR221GLFS/401-1427-1-ND/550466?WT.z_cid=ref_snapeda&utm_source=snapeda&utm_medium=aggregator&utm_campaign=buynow" H 3750 6300 50  0001 L BNN "Field7"
-F 8 "SWITCH TACTILE SPST-NO 0.05A 32V" H 3750 6300 50  0001 L BNN "Field8"
-	1    3750 6300
-	0    -1   -1   0
-$EndComp
-$Comp
-L KMR221GLFS BOTTOM_RST2
-U 1 1 5A4E75A7
-P 4550 6650
-F 0 "BOTTOM_RST2" H 4450 6740 50  0000 L BNN
-F 1 "KMR221GLFS" H 4440 6400 50  0000 L BNN
-F 2 "SW_KMR221GLFS" H 4550 6650 50  0001 L BNN
-F 3 "401-1427-1-ND" H 4550 6650 50  0001 L BNN
-F 4 "C&K Components" H 4550 6650 50  0001 L BNN "Field4"
-F 5 "None" H 4550 6650 50  0001 L BNN "Field5"
-F 6 "KMR221GLFS" H 4550 6650 50  0001 L BNN "Field6"
-F 7 "https://www.digikey.com.mx/product-detail/en/c-k/KMR221GLFS/401-1427-1-ND/550466?WT.z_cid=ref_snapeda&utm_source=snapeda&utm_medium=aggregator&utm_campaign=buynow" H 4550 6650 50  0001 L BNN "Field7"
-F 8 "SWITCH TACTILE SPST-NO 0.05A 32V" H 4550 6650 50  0001 L BNN "Field8"
-	1    4550 6650
-	0    -1   -1   0
+L +3.3V #PWR035
+U 1 1 5A4EAA4E
+P 6600 950
+F 0 "#PWR035" H 6600 800 50  0001 C CNN
+F 1 "+3.3V" H 6600 1090 50  0000 C CNN
+F 2 "" H 6600 950 50  0001 C CNN
+F 3 "" H 6600 950 50  0001 C CNN
+	1    6600 950
+	1    0    0    -1
+$EndComp
+Text Label 4200 1500 0    60   ~ 0
+SCL
+$Comp
+L +3.3V #PWR036
+U 1 1 5A4F3DF1
+P 4450 1150
+F 0 "#PWR036" H 4450 1000 50  0001 C CNN
+F 1 "+3.3V" H 4450 1290 50  0000 C CNN
+F 2 "" H 4450 1150 50  0001 C CNN
+F 3 "" H 4450 1150 50  0001 C CNN
+	1    4450 1150
+	1    0    0    -1
+$EndComp
+$Comp
+L B3U-1000P S?
+U 1 1 5A50A6C4
+P 3750 6850
+F 0 "S?" H 3449 7050 50  0000 L BNN
+F 1 "BOTTON_BOOT" H 3449 6549 50  0000 L BNN
+F 2 "SW_B3U-1000P" H 3750 6850 50  0001 L BNN
+F 3 "SWITCH TACTILE SPST-NO 0.05A 12V" H 3750 6850 50  0001 L BNN
+F 4 "None" H 3750 6850 50  0001 L BNN "Field4"
+F 5 "Omron" H 3750 6850 50  0001 L BNN "Field5"
+F 6 "SW1020CT-ND" H 3750 6850 50  0001 L BNN "Field6"
+F 7 "https://www.digikey.com.mx/product-detail/en/omron-electronics-inc-emc-div/B3U-1000P/SW1020CT-ND/1534357?WT.z_cid=ref_snapeda&utm_source=snapeda&utm_medium=aggregator&utm_campaign=buynow" H 3750 6850 50  0001 L BNN "Field7"
+F 8 "B3U-1000P" H 3750 6850 50  0001 L BNN "Field8"
+	1    3750 6850
+	0    1    1    0
+$EndComp
+$Comp
+L B3U-1000P S?
+U 1 1 5A50AFF2
+P 4500 6850
+F 0 "S?" H 4199 7050 50  0000 L BNN
+F 1 "BOTTON_RST" H 4199 6549 50  0000 L BNN
+F 2 "SW_B3U-1000P" H 4500 6850 50  0001 L BNN
+F 3 "SWITCH TACTILE SPST-NO 0.05A 12V" H 4500 6850 50  0001 L BNN
+F 4 "None" H 4500 6850 50  0001 L BNN "Field4"
+F 5 "Omron" H 4500 6850 50  0001 L BNN "Field5"
+F 6 "SW1020CT-ND" H 4500 6850 50  0001 L BNN "Field6"
+F 7 "https://www.digikey.com.mx/product-detail/en/omron-electronics-inc-emc-div/B3U-1000P/SW1020CT-ND/1534357?WT.z_cid=ref_snapeda&utm_source=snapeda&utm_medium=aggregator&utm_campaign=buynow" H 4500 6850 50  0001 L BNN "Field7"
+F 8 "B3U-1000P" H 4500 6850 50  0001 L BNN "Field8"
+	1    4500 6850
+	0    1    1    0
 $EndComp
 Wire Wire Line
@@
 	2650 6700 2650 6450
 Wire Wire Line
-	4700 1500 4900 1500
-Wire Wire Line
-	6300 1300 6500 1300
-Wire Wire Line
-	6800 1300 6950 1300
-Wire Wire Line
-	4400 1500 4250 1500
+	4200 1500 4900 1500
 Wire Wire Line
 	4800 1800 4800 1950
@@
 Wire Wire Line
 	7100 4200 8000 4200
-Connection ~ 7100 4850
 Wire Wire Line
 	8200 4200 8400 4200
@@
 Wire Wire Line
 	5650 5950 5650 6950
-Wire Wire Line
-	3750 6850 3750 6600
-Wire Wire Line
-	4550 5150 4550 5650
 Wire Wire Line
 	4950 5950 4950 6950
@@
 	3350 2600 3350 3100
 Wire Wire Line
-	3750 5150 3750 6000
-Wire Wire Line
-	4550 5950 4550 6350
-$Comp
-L GND #PWR035
-U 1 1 5A4E9AF2
-P 4100 6050
-F 0 "#PWR035" H 4100 5800 50  0001 C CNN
-F 1 "GND" H 4100 5900 50  0000 C CNN
-F 2 "" H 4100 6050 50  0001 C CNN
-F 3 "" H 4100 6050 50  0001 C CNN
-	1    4100 6050
-	1    0    0    -1
-$EndComp
-$Comp
-L GND #PWR036
-U 1 1 5A4E9B5E
-P 4850 6350
-F 0 "#PWR036" H 4850 6100 50  0001 C CNN
-F 1 "GND" H 4850 6200 50  0000 C CNN
-F 2 "" H 4850 6350 50  0001 C CNN
-F 3 "" H 4850 6350 50  0001 C CNN
-	1    4850 6350
-	1    0    0    -1
-$EndComp
-Wire Wire Line
-	3850 6000 3850 5900
-Wire Wire Line
-	3850 5900 4100 5900
-Wire Wire Line
-	4100 5900 4100 6050
-Wire Wire Line
-	4650 6350 4650 6250
-Wire Wire Line
-	4650 6250 4850 6250
-Wire Wire Line
-	4850 6250 4850 6350
+	3750 5150 3750 6350
+Wire Wire Line
+	4450 1450 4450 1500
+Connection ~ 4450 1500
+Wire Wire Line
+	6600 1250 6600 1300
+Connection ~ 6600 1300
+Wire Wire Line
+	6300 1300 6800 1300
+Wire Wire Line
+	4500 5950 4500 6350
+Wire Wire Line
+	4500 5150 4500 5650
+Wire Wire Line
+	3750 7450 3750 7350
 $EndSCHEMATC

Commit message: VCC
Etiqueta VCC y VCC ESP cambiado por 3.3
Connections:
- wire segments 144 -> 147
Changed lines of the file:
@@
 	1    0    0    -1
 $EndComp
-Text Label 7250 2100 0    60   ~ 0
-VCC
 Text Label 7750 2100 0    60   ~ 0
 BAT
@@
 	1    0    0    -1
 $EndComp
-Text Label 6600 4500 0    60   ~ 0
-VCC
 $Comp
 L GND #PWR021
@@
 	1    0    0    -1
 $EndComp
-Text Label 6450 3900 0    60   ~ 0
-VCC
 $Comp
 L D_Schottky D4
@@
 NoConn ~ 4800 3200
 NoConn ~ 3500 8600
-Text Label 3700 4250 0    60   ~ 0
-VCC
 Text Label 3950 4250 0    60   ~ 0
 D1
@@
 Connection ~ 2650 1350
 Wire Wire Line
-	7100 4850 8300 4850
-Wire Wire Line
-	7100 4200 8000 4200
-Wire Wire Line
 	8200 4200 8400 4200
 Wire Wire Line
@@
 Connection ~ 10300 5050
 Wire Wire Line
-	4900 1300 3950 1300
-Wire Wire Line
-	3950 1300 3950 1400
+	3950 900  3950 1400
 Wire Wire Line
 	3950 1700 3950 1800
@@
 	4100 3800 4100 3700
 Wire Wire Line
-	3700 4250 3700 3850
-Wire Wire Line
 	3700 3850 4200 3850
 Wire Wire Line
@@
 Wire Wire Line
 	6700 3500 6600 3500
-Wire Wire Line
-	6450 3900 6450 3500
 Wire Wire Line
 	6450 3500 6400 3500
@@
 	5300 5650 5300 5150
 Wire Wire Line
-	7100 4200 7100 4850
-Wire Wire Line
-	6600 4500 7100 4500
-Connection ~ 7100 4500
-Wire Wire Line
 	1300 1500 1300 1350
 Wire Wire Line
@@
 Wire Wire Line
 	3750 7450 3750 7350
+$Comp
+L +3.3V #PWR?
+U 1 1 5A51A868
+P 3700 4150
+F 0 "#PWR?" H 3700 4000 50  0001 C CNN
+F 1 "+3.3V" H 3700 4290 50  0000 C CNN
+F 2 "" H 3700 4150 50  0001 C CNN
+F 3 "" H 3700 4150 50  0001 C CNN
+	1    3700 4150
+	-1   0    0    1
+$EndComp
+Wire Wire Line
+	3700 3850 3700 4150
+$Comp
+L VCC #PWR?
+U 1 1 5A51CA39
+P 7600 4550
+F 0 "#PWR?" H 7600 4400 50  0001 C CNN
+F 1 "VCC" H 7600 4700 50  0000 C CNN
+F 2 "" H 7600 4550 50  0001 C CNN
+F 3 "" H 7600 4550 50  0001 C CNN
+	1    7600 4550
+	0    -1   -1   0
+$EndComp
+$Comp
+L VCC #PWR?
+U 1 1 5A51CAA5
+P 6500 3800
+F 0 "#PWR?" H 6500 3650 50  0001 C CNN
+F 1 "VCC" H 6500 3950 50  0000 C CNN
+F 2 "" H 6500 3800 50  0001 C CNN
+F 3 "" H 6500 3800 50  0001 C CNN
+	1    6500 3800
+	-1   0    0    1
+$EndComp
+$Comp
+L VCC #PWR?
+U 1 1 5A51D5B9
+P 7250 2100
+F 0 "#PWR?" H 7250 1950 50  0001 C CNN
+F 1 "VCC" H 7250 2250 50  0000 C CNN
+F 2 "" H 7250 2100 50  0001 C CNN
+F 3 "" H 7250 2100 50  0001 C CNN
+	1    7250 2100
+	1    0    0    -1
+$EndComp
+Wire Wire Line
+	6450 3500 6450 3700
+Wire Wire Line
+	6450 3700 6500 3700
+Wire Wire Line
+	6500 3700 6500 3800
+Wire Wire Line
+	7600 4850 8300 4850
+Wire Wire Line
+	7600 4200 7600 4850
+Wire Wire Line
+	8000 4200 7600 4200
+Connection ~ 7600 4550
+Wire Wire Line
+	4900 1300 4650 1300
+Wire Wire Line
+	4650 1300 4650 900
+Wire Wire Line
+	4650 900  3950 900
 $EndSCHEMATC

Commit message: ADAP_MEDIDAS
Adaptador del ESP8266 para programación. Y modificacion del esquematico placa principal para el adaptador.
Parts:
- removed J4: ADAP_ESP, Pin_Headers:Pin_Header_Straight_2x08_Pitch2.54mm, symbol Conn_02x08_Top_Bottom
- removed R10, R12, R18, R9: 10K, Resistors_SMD:R_0603, symbol R
- removed R11, R13: 4.7K, Resistors_SMD:R_0603, symbol R
- added J1: ADAP_ESP, Pin_Headers:Pin_Header_Straight_2x06_Pitch2.54mm, symbol Conn_02x06_Odd_Even
- BTRTC1: value 3.3V -> 3.3Va; footprint Battery_Holders:Keystone_1058_1x2032-CoinCell -> PADS:Keystone_battery; Fieldname (none) -> Value
- C1, C2, C3: footprint Capacitors_SMD:C_0603 -> Capacitors_SMD:C_0805
- COMUN1, COMUN2, IN1, IN2: footprint PADS:PAD_5x3mm -> PADS:Pad_5x3mm_45
- D1, D2: footprint LEDs:LED_0603 -> LEDs:LED_0805
- D3, D4: value RB161 -> NRVB120
- R1, R14, R15, R16, R17, R2, R3, R4, R5, R6, R7, R8: footprint Resistors_SMD:R_0603 -> Resistors_SMD:R_0805
- S1: renamed from S?; value BOTTON_BOOT -> BOTTOM_BOOT; footprint SW_B3U-1000P -> B3U-1000P:SW_B3U-1000P
- S2: renamed from S?; value BOTTON_RST -> BOTTOM_RST; footprint SW_B3U-1000P -> B3U-1000P:SW_B3U-1000P
- U1, U2, U3, U4: footprint Housings_DIP:DIP-6_W7.62mm -> Housings_DIP:DIP-6_W7.62mm_SMDSocket_SmallPads
- U6: footprint TO_SOT_Packages_SMD:SOT-223-3Lead_TabPin2 -> TO_SOT_Packages_SMD:SOT-223-3_TabPin2
Connections:
- net labels removed: CH, GPIO15, GPIO2
- wire segments 147 -> 129
- no-connect marks 10 -> 9
Other:
- moved on the sheet: S1, S2

Commit message: PCBS_Adap_mon
Correxión del RX y TX del adaptador, PCB monitor doble capa.
Parts:
- C1, C2, C3: footprint Capacitors_SMD:C_0805 -> Capacitors_SMD:C_0805_HandSoldering
- COMUN1, COMUN2, IN1, IN2: footprint PADS:Pad_5x3mm_45 -> PADS:PAD_5x3mm
- D1, D2: footprint LEDs:LED_0805 -> LEDs:LED_0805_HandSoldering
- R1, R14, R15, R16, R17, R2, R3, R4, R5, R6, R7, R8: footprint Resistors_SMD:R_0805 -> Resistors_SMD:R_0805_HandSoldering
Changed lines of the file:
@@
 F 0 "R6" V 2730 1650 50  0000 C CNN
 F 1 "10K" V 2650 1650 50  0000 C CNN
-F 2 "Resistors_SMD:R_0805" V 2580 1650 50  0001 C CNN
+F 2 "Resistors_SMD:R_0805_HandSoldering" V 2580 1650 50  0001 C CNN
 F 3 "" H 2650 1650 50  0001 C CNN
 	1    2650 1650
@@
 F 0 "R2" V 1380 2700 50  0000 C CNN
 F 1 "2K" V 1300 2700 50  0000 C CNN
-F 2 "Resistors_SMD:R_0805" V 1230 2700 50  0001 C CNN
+F 2 "Resistors_SMD:R_0805_HandSoldering" V 1230 2700 50  0001 C CNN
 F 3 "" H 1300 2700 50  0001 C CNN
 F 4 "Value" H 1300 2700 60  0001 C CNN "Fieldname"
@@
 F 0 "R7" V 2730 3150 50  0000 C CNN
 F 1 "10K" V 2650 3150 50  0000 C CNN
-F 2 "Resistors_SMD:R_0805" V 2580 3150 50  0001 C CNN
+F 2 "Resistors_SMD:R_0805_HandSoldering" V 2580 3150 50  0001 C CNN
 F 3 "" H 2650 3150 50  0001 C CNN
 	1    2650 3150
@@
 F 0 "R1" V 1330 4350 50  0000 C CNN
 F 1 "2K" V 1250 4350 50  0000 C CNN
-F 2 "Resistors_SMD:R_0805" V 1180 4350 50  0001 C CNN
+F 2 "Resistors_SMD:R_0805_HandSoldering" V 1180 4350 50  0001 C CNN
 F 3 "" H 1250 4350 50  0001 C CNN
 	1    1250 4350
@@
 F 0 "R5" V 2680 4800 50  0000 C CNN
 F 1 "10K" V 2600 4800 50  0000 C CNN
-F 2 "Resistors_SMD:R_0805" V 2530 4800 50  0001 C CNN
+F 2 "Resistors_SMD:R_0805_HandSoldering" V 2530 4800 50  0001 C CNN
 F 3 "" H 2600 4800 50  0001 C CNN
 	1    2600 4800
@@
 F 0 "R3" V 1380 5900 50  0000 C CNN
 F 1 "2K" V 1300 5900 50  0000 C CNN
-F 2 "Resistors_SMD:R_0805" V 1230 5900 50  0001 C CNN
+F 2 "Resistors_SMD:R_0805_HandSoldering" V 1230 5900 50  0001 C CNN
 F 3 "" H 1300 5900 50  0001 C CNN
 	1    1300 5900
@@
 F 0 "R8" V 2730 6300 50  0000 C CNN
 F 1 "10K" V 2650 6300 50  0000 C CNN
-F 2 "Resistors_SMD:R_0805" V 2580 6300 50  0001 C CNN
+F 2 "Resistors_SMD:R_0805_HandSoldering" V 2580 6300 50  0001 C CNN
 F 3 "" H 2650 6300 50  0001 C CNN
 	1    2650 6300
@@
 F 0 "R4" V 1430 1150 50  0000 C CNN
 F 1 "2K" V 1350 1150 50  0000 C CNN
-F 2 "Resistors_SMD:R_0805" V 1280 1150 50  0001 C CNN
+F 2 "Resistors_SMD:R_0805_HandSoldering" V 1280 1150 50  0001 C CNN
 F 3 "" H 1350 1150 50  0001 C CNN
 	1    1350 1150
@@
 F 0 "IN1" H 850 1250 50  0000 C CNN
 F 1 "0_IN" H 850 1050 50  0000 C CNN
-F 2 "PADS:Pad_5x3mm_45" H 850 1150 50  0001 C CNN
+F 2 "PADS:PAD_5x3mm" H 850 1150 50  0001 C CNN
 F 3 "" H 850 1150 50  0001 C CNN
 	1    850  1150
@@
 F 0 "IN2" H 750 2800 50  0000 C CNN
 F 1 "1_IN" H 750 2600 50  0000 C CNN
-F 2 "PADS:Pad_5x3mm_45" H 750 2700 50  0001 C CNN
+F 2 "PADS:PAD_5x3mm" H 750 2700 50  0001 C CNN
 F 3 "" H 750 2700 50  0001 C CNN
 	1    750  2700
@@
 F 0 "COMUN1" H 850 7600 50  0000 C CNN
 F 1 "NC" H 850 7400 50  0000 C CNN
-F 2 "PADS:Pad_5x3mm_45" H 850 7500 50  0001 C CNN
+F 2 "PADS:PAD_5x3mm" H 850 7500 50  0001 C CNN
 F 3 "" H 850 7500 50  0001 C CNN
 	1    850  7500
@@
 F 0 "COMUN2" H 850 6900 50  0000 C CNN
 F 1 "TORRETA" H 850 6700 50  0000 C CNN
-F 2 "PADS:Pad_5x3mm_45" H 850 6800 50  0001 C CNN
+F 2 "PADS:PAD_5x3mm" H 850 6800 50  0001 C CNN
 F 3 "" H 850 6800 50  0001 C CNN
 	1    850  6800
@@
 F 0 "D2" H 8050 4325 50  0000 L CNN
 F 1 "LED_CHAR" H 7925 4100 50  0000 L CNN
-F 2 "LEDs:LED_0805" V 8100 4200 50  0001 C CNN
+F 2 "LEDs:LED_0805_HandSoldering" V 8100 4200 50  0001 C CNN
 F 3 "" V 8100 4200 50  0001 C CNN
 	1    8100 4200
@@
 F 0 "R15" V 8630 4200 50  0000 C CNN
 F 1 "1K" V 8550 4200 50  0000 C CNN
-F 2 "Resistors_SMD:R_0805" V 8480 4200 50  0001 C CNN
+F 2 "Resistors_SMD:R_0805_HandSoldering" V 8480 4200 50  0001 C CNN
 F 3 "" H 8550 4200 50  0001 C CNN
 	1    8550 4200
@@
 F 0 "R14" V 7980 5150 50  0000 C CNN
 F 1 "10K" V 7900 5150 50  0000 C CNN
-F 2 "Resistors_SMD:R_0805" V 7830 5150 50  0001 C CNN
+F 2 "Resistors_SMD:R_0805_HandSoldering" V 7830 5150 50  0001 C CNN
 F 3 "" H 7900 5150 50  0001 C CNN
 	1    7900 5150
@@
 F 0 "C2" H 10310 5320 50  0000 L CNN
 F 1 "10u" H 10310 5170 50  0000 L CNN
-F 2 "Capacitors_SMD:C_0805" H 10300 5250 50  0001 C CNN
+F 2 "Capacitors_SMD:C_0805_HandSoldering" H 10300 5250 50  0001 C CNN
 F 3 "" H 10300 5250 50  0001 C CNN
 	1    10300 5250
@@
 F 0 "R16" V 10080 5050 50  0000 C CNN
 F 1 "10K" V 10000 5050 50  0000 C CNN
-F 2 "Resistors_SMD:R_0805" V 9930 5050 50  0001 C CNN
+F 2 "Resistors_SMD:R_0805_HandSoldering" V 9930 5050 50  0001 C CNN
 F 3 "" H 10000 5050 50  0001 C CNN
 	1    10000 5050
@@
 F 0 "C1" H 8160 3020 50  0000 L CNN
 F 1 "2.2u" H 8160 2870 50  0000 L CNN
-F 2 "Capacitors_SMD:C_0805" H 8150 2950 50  0001 C CNN
+F 2 "Capacitors_SMD:C_0805_HandSoldering" H 8150 2950 50  0001 C CNN
 F 3 "" H 8150 2950 50  0001 C CNN
 	1    8150 2950
@@
 F 0 "C3" H 9360 2970 50  0000 L CNN
 F 1 "4.7u" H 9360 2820 50  0000 L CNN
-F 2 "Capacitors_SMD:C_0805" H 9350 2900 50  0001 C CNN
+F 2 "Capacitors_SMD:C_0805_HandSoldering" H 9350 2900 50  0001 C CNN
 F 3 "" H 9350 2900 50  0001 C CNN
 	1    9350 2900
@@
 F 0 "R17" V 10480 2950 50  0000 C CNN
 F 1 "1K" V 10400 2950 50  0000 C CNN
-F 2 "Resistors_SMD:R_0805" V 10330 2950 50  0001 C CNN
+F 2 "Resistors_SMD:R_0805_HandSoldering" V 10330 2950 50  0001 C CNN
 F 3 "" H 10400 2950 50  0001 C CNN
 	1    10400 2950
@@
 F 0 "D1" H 10350 2625 50  0000 L CNN
 F 1 "LED_ON" H 10225 2400 50  0000 L CNN
-F 2 "LEDs:LED_0805" V 10400 2500 50  0001 C CNN
+F 2 "LEDs:LED_0805_HandSoldering" V 10400 2500 50  0001 C CNN
 F 3 "" V 10400 2500 50  0001 C CNN
 	1    10400 2500

Commit message: Tracks fix
Parts:
- U1, U2, U3, U4: symbol 4N25 -> 4N25-RESCUE-WiFiMonitor
Changed lines of the file:
@@
 EESchema Schematic File Version 2
+LIBS:WiFiMonitor-rescue
 LIBS:power
 LIBS:device
@@
 LIBS:contrib
 LIBS:valves
-LIBS:MCP73831T-4ADI_OT
-LIBS:B3U-1000P
 LIBS:WiFiMonitor-cache
 EELAYER 25 0
@@
 $EndDescr
 $Comp
-L 4N25 U2
+L 4N25-RESCUE-WiFiMonitor U2
 U 1 1 5A45C686
 P 1900 1250
@@
 $EndComp
 $Comp
-L 4N25 U3
+L 4N25-RESCUE-WiFiMonitor U3
 U 1 1 5A49A2CF
 P 1900 2800
@@
 $EndComp
 $Comp
-L 4N25 U1
+L 4N25-RESCUE-WiFiMonitor U1
 U 1 1 5A49B2B9
 P 1850 4450
@@
 $EndComp
 $Comp
-L 4N25 U4
+L 4N25-RESCUE-WiFiMonitor U4
 U 1 1 5A49B3A4
 P 1900 6000
