File: Hardware/WiFiMonitor.sch (KiCad schematic (older format))
At the start: 38 parts, among them J1 ADAP_ESP, J3 BATT, J5 FTDI, U1 4N25, U2 4N25, U3 4N25, U4 4N25, U5 MCP73831T-4ADI/OT, U6 AP1117-33, U7 DS3231MZ+

Commit message: PADS_TH
Pads de los voltajes de entradas en Through-Hole y espacio para el tornillo en el centro,
Parts:
- COMUN1, COMUN2, IN1, IN2, IN3, IN4: footprint PADS:PAD_5x3mm -> PADS:PAD_4X2mmTH
Changed lines of the file:
@@
 LIBS:contrib
 LIBS:valves
+LIBS:MCP73831T-4ADI_OT
+LIBS:B3U-1000P
 LIBS:WiFiMonitor-cache
 EELAYER 25 0
@@
 F 0 "IN1" H 850 1250 50  0000 C CNN
 F 1 "0_IN" H 850 1050 50  0000 C CNN
-F 2 "PADS:PAD_5x3mm" H 850 1150 50  0001 C CNN
+F 2 "PADS:PAD_4X2mmTH" H 850 1150 50  0001 C CNN
 F 3 "" H 850 1150 50  0001 C CNN
 	1    850  1150
@@
 F 0 "IN2" H 750 2800 50  0000 C CNN
 F 1 "1_IN" H 750 2600 50  0000 C CNN
-F 2 "PADS:PAD_5x3mm" H 750 2700 50  0001 C CNN
+F 2 "PADS:PAD_4X2mmTH" H 750 2700 50  0001 C CNN
 F 3 "" H 750 2700 50  0001 C CNN
 	1    750  2700
@@
 F 0 "IN3" H 750 4450 50  0000 C CNN
 F 1 "2_IN" H 750 4250 50  0000 C CNN
-F 2 "PADS:PAD_5x3mm" H 750 4350 50  0001 C CNN
+F 2 "PADS:PAD_4X2mmTH" H 750 4350 50  0001 C CNN
 F 3 "" H 750 4350 50  0001 C CNN
 	1    750  4350
@@
 F 0 "IN4" H 800 6000 50  0000 C CNN
 F 1 "3_IN" H 800 5800 50  0000 C CNN
-F 2 "PADS:PAD_5x3mm" H 800 5900 50  0001 C CNN
+F 2 "PADS:PAD_4X2mmTH" H 800 5900 50  0001 C CNN
 F 3 "" H 800 5900 50  0001 C CNN
 	1    800  5900
@@
 F 0 "COMUN1" H 850 7600 50  0000 C CNN
 F 1 "NC" H 850 7400 50  0000 C CNN
-F 2 "PADS:PAD_5x3mm" H 850 7500 50  0001 C CNN
+F 2 "PADS:PAD_4X2mmTH" H 850 7500 50  0001 C CNN
 F 3 "" H 850 7500 50  0001 C CNN
 	1    850  7500
@@
 F 0 "COMUN2" H 850 6900 50  0000 C CNN
 F 1 "TORRETA" H 850 6700 50  0000 C CNN
-F 2 "PADS:PAD_5x3mm" H 850 6800 50  0001 C CNN
+F 2 "PADS:PAD_4X2mmTH" H 850 6800 50  0001 C CNN
 F 3 "" H 850 6800 50  0001 C CNN
 	1    850  6800
