File: Hardware/WiFiMonitor.sch (KiCad schematic (older format))
At the start: 40 parts, among them J1 ADAP_ESP, J2 FTDI, J3 BATT, U1 4N25, U2 4N25, U3 4N25, U4 4N25, U5 MCP73831T-4ADI/OT, U6 AP1117-33, U7 DS3231MZ+

Commit message: changes charger sch
Parts:
- removed R16: 10K, Resistors_SMD:R_0805_HandSoldering, symbol R
- added C6: 4.7u, symbol C
- R14: value 10K -> 1K
Connections:
- net BAT: now also U5.3 (VBAT)
- net GND: now also C6.2
- net VCC: now also C6.1
Changed lines of the file:
@@
 LIBS:contrib
 LIBS:valves
-LIBS:MCP73831T-4ADI_OT
-LIBS:B3U-1000P
 LIBS:WiFiMonitor-cache
 EELAYER 25 0
@@
 $EndComp
 $Comp
-L GND #PWR01
+L GND #PWR12
 U 1 1 5A45CFEC
 P 2650 2000
-F 0 "#PWR01" H 2650 1750 50  0001 C CNN
+F 0 "#PWR12" H 2650 1750 50  0001 C CNN
 F 1 "GND" H 2650 1850 50  0000 C CNN
 F 2 "" H 2650 2000 50  0001 C CNN
@@
 $EndComp
 $Comp
-L GND #PWR02
+L GND #PWR13
 U 1 1 5A49D5FF
 P 2650 3500
-F 0 "#PWR02" H 2650 3250 50  0001 C CNN
+F 0 "#PWR13" H 2650 3250 50  0001 C CNN
 F 1 "GND" H 2650 3350 50  0000 C CNN
 F 2 "" H 2650 3500 50  0001 C CNN
@@
 $EndComp
 $Comp
-L GND #PWR03
+L GND #PWR11
 U 1 1 5A49D66B
 P 2600 5250
-F 0 "#PWR03" H 2600 5000 50  0001 C CNN
+F 0 "#PWR11" H 2600 5000 50  0001 C CNN
 F 1 "GND" H 2600 5100 50  0000 C CNN
 F 2 "" H 2600 5250 50  0001 C CNN
@@
 $EndComp
 $Comp
-L GND #PWR04
+L GND #PWR14
 U 1 1 5A49D6D7
 P 2650 6700
-F 0 "#PWR04" H 2650 6450 50  0001 C CNN
+F 0 "#PWR14" H 2650 6450 50  0001 C CNN
 F 1 "GND" H 2650 6550 50  0000 C CNN
 F 2 "" H 2650 6700 50  0001 C CNN
@@
 $EndComp
 $Comp
-L GND #PWR05
+L GND #PWR20
 U 1 1 5A4A8EE5
 P 4800 1850
-F 0 "#PWR05" H 4800 1600 50  0001 C CNN
+F 0 "#PWR20" H 4800 1600 50  0001 C CNN
 F 1 "GND" H 4800 1700 50  0000 C CNN
 F 2 "" H 4800 1850 50  0001 C CNN
@@
 $EndComp
 $Comp
-L +3.3V #PWR06
+L +3.3V #PWR10
 U 1 1 5A4AF41B
 P 2600 900
-F 0 "#PWR06" H 2600 750 50  0001 C CNN
+F 0 "#PWR10" H 2600 750 50  0001 C CNN
 F 1 "+3.3V" H 2600 1040 50  0000 C CNN
 F 2 "" H 2600 900 50  0001 C CNN
@@
 $EndComp
 $Comp
-L +3.3V #PWR07
+L +3.3V #PWR8
 U 1 1 5A4AF460
 P 2550 2500
-F 0 "#PWR07" H 2550 2350 50  0001 C CNN
+F 0 "#PWR8" H 2550 2350 50  0001 C CNN
 F 1 "+3.3V" H 2550 2640 50  0000 C CNN
 F 2 "" H 2550 2500 50  0001 C CNN
@@
 $EndComp
 $Comp
-L +3.3V #PWR08
+L +3.3V #PWR7
 U 1 1 5A4AF48F
 P 2500 4100
-F 0 "#PWR08" H 2500 3950 50  0001 C CNN
+F 0 "#PWR7" H 2500 3950 50  0001 C CNN
 F 1 "+3.3V" H 2500 4240 50  0000 C CNN
 F 2 "" H 2500 4100 50  0001 C CNN
@@
 $EndComp
 $Comp
-L +3.3V #PWR09
+L +3.3V #PWR9
 U 1 1 5A4AF4D4
 P 2550 5750
-F 0 "#PWR09" H 2550 5600 50  0001 C CNN
+F 0 "#PWR9" H 2550 5600 50  0001 C CNN
 F 1 "+3.3V" H 2550 5890 50  0000 C CNN
 F 2 "" H 2550 5750 50  0001 C CNN
@@
 $EndComp
 $Comp
-L +3.3V #PWR010
+L +3.3V #PWR19
 U 1 1 5A4B1476
 P 4800 1100
-F 0 "#PWR010" H 4800 950 50  0001 C CNN
+F 0 "#PWR19" H 4800 950 50  0001 C CNN
 F 1 "+3.3V" H 4800 1240 50  0000 C CNN
 F 2 "" H 4800 1100 50  0001 C CNN
@@
 P 7900 5150
 F 0 "R14" V 7980 5150 50  0000 C CNN
-F 1 "10K" V 7900 5150 50  0000 C CNN
+F 1 "1K" V 7900 5150 50  0000 C CNN
 F 2 "Resistors_SMD:R_0805_HandSoldering" V 7830 5150 50  0001 C CNN
 F 3 "" H 7900 5150 50  0001 C CNN
@@
 	1    10300 5250
 	1    0    0    -1
-$EndComp
-$Comp
-L R R16
-U 1 1 5A4C77E5
-P 10000 5050
-F 0 "R16" V 10080 5050 50  0000 C CNN
-F 1 "10K" V 10000 5050 50  0000 C CNN
-F 2 "Resistors_SMD:R_0805_HandSoldering" V 9930 5050 50  0001 C CNN
-F 3 "" H 10000 5050 50  0001 C CNN
-	1    10000 5050
-	0    1    1    0
 $EndComp
 $Comp
@@
 $EndComp
 $Comp
-L GND #PWR011
+L GND #PWR27
 U 1 1 5A4C8277
 P 7900 5650
-F 0 "#PWR011" H 7900 5400 50  0001 C CNN
+F 0 "#PWR27" H 7900 5400 50  0001 C CNN
 F 1 "GND" H 7900 5500 50  0000 C CNN
 F 2 "" H 7900 5650 50  0001 C CNN
@@
 $EndComp
 $Comp
-L GND #PWR012
+L GND #PWR33
 U 1 1 5A4C87C8
 P 10300 5550
-F 0 "#PWR012" H 10300 5300 50  0001 C CNN
+F 0 "#PWR33" H 10300 5300 50  0001 C CNN
 F 1 "GND" H 10300 5400 50  0000 C CNN
 F 2 "" H 10300 5550 50  0001 C CNN
@@
 $EndComp
 $Comp
-L GND #PWR013
+L GND #PWR29
 U 1 1 5A4D1767
 P 8750 3250
-F 0 "#PWR013" H 8750 3000 50  0001 C CNN
+F 0 "#PWR29" H 8750 3000 50  0001 C CNN
 F 1 "GND" H 8750 3100 50  0000 C CNN
 F 2 "" H 8750 3250 50  0001 C CNN
@@
 $EndComp
 $Comp
-L +3.3V #PWR014
+L +3.3V #PWR32
 U 1 1 5A4D19E5
 P 9600 2350
-F 0 "#PWR014" H 9600 2200 50  0001 C CNN
+F 0 "#PWR32" H 9600 2200 50  0001 C CNN
 F 1 "+3.3V" H 9600 2490 50  0000 C CNN
 F 2 "" H 9600 2350 50  0001 C CNN
@@
 BAT
 $Comp
-L GND #PWR015
+L GND #PWR30
 U 1 1 5A4D5453
 P 9150 1250
-F 0 "#PWR015" H 9150 1000 50  0001 C CNN
+F 0 "#PWR30" H 9150 1000 50  0001 C CNN
 F 1 "GND" H 9150 1100 50  0000 C CNN
 F 2 "" H 9150 1250 50  0001 C CNN
@@
 $EndComp
 $Comp
-L GND #PWR016
+L GND #PWR16
 U 1 1 5A4D8876
 P 3800 4200
-F 0 "#PWR016" H 3800 3950 50  0001 C CNN
+F 0 "#PWR16" H 3800 3950 50  0001 C CNN
 F 1 "GND" H 3800 4050 50  0000 C CNN
 F 2 "" H 3800 4200 50  0001 C CNN
@@
 RST
 $Comp
-L GND #PWR017
+L GND #PWR21
 U 1 1 5A4C5C3E
 P 5300 6800
-F 0 "#PWR017" H 5300 6550 50  0001 C CNN
+F 0 "#PWR21" H 5300 6550 50  0001 C CNN
 F 1 "GND" H 5300 6650 50  0000 C CNN
 F 2 "" H 5300 6800 50  0001 C CNN
@@
 $EndComp
 $Comp
-L GND #PWR018
+L GND #PWR28
 U 1 1 5A4E1946
 P 8150 3250
-F 0 "#PWR018" H 8150 3000 50  0001 C CNN
+F 0 "#PWR28" H 8150 3000 50  0001 C CNN
 F 1 "GND" H 8150 3100 50  0000 C CNN
 F 2 "" H 8150 3250 50  0001 C CNN
@@
 $EndComp
 $Comp
-L GND #PWR019
+L GND #PWR31
 U 1 1 5A4E1A3F
 P 9350 3250
-F 0 "#PWR019" H 9350 3000 50  0001 C CNN
+F 0 "#PWR31" H 9350 3000 50  0001 C CNN
 F 1 "GND" H 9350 3100 50  0000 C CNN
 F 2 "" H 9350 3250 50  0001 C CNN
@@
 $EndComp
 $Comp
-L GND #PWR020
+L GND #PWR18
 U 1 1 5A4FDC73
 P 4550 6800
-F 0 "#PWR020" H 4550 6550 50  0001 C CNN
+F 0 "#PWR18" H 4550 6550 50  0001 C CNN
 F 1 "GND" H 4550 6650 50  0000 C CNN
 F 2 "" H 4550 6800 50  0001 C CNN
@@
 RX
 $Comp
-L GND #PWR021
+L GND #PWR23
 U 1 1 5A50C999
 P 6700 3800
-F 0 "#PWR021" H 6700 3550 50  0001 C CNN
+F 0 "#PWR23" H 6700 3550 50  0001 C CNN
 F 1 "GND" H 6700 3650 50  0000 C CNN
 F 2 "" H 6700 3800 50  0001 C CNN
@@
 NoConn ~ 6500 3500
 $Comp
-L GNDA #PWR022
+L GNDA #PWR4
 U 1 1 5A57ECC2
 P 1300 3050
-F 0 "#PWR022" H 1300 2800 50  0001 C CNN
+F 0 "#PWR4" H 1300 2800 50  0001 C CNN
 F 1 "GNDA" H 1300 2900 50  0000 C CNN
 F 2 "" H 1300 3050 50  0001 C CNN
@@
 $EndComp
 $Comp
-L GNDA #PWR023
+L GNDA #PWR3
 U 1 1 5A58195E
 P 1300 1500
-F 0 "#PWR023" H 1300 1250 50  0001 C CNN
+F 0 "#PWR3" H 1300 1250 50  0001 C CNN
 F 1 "GNDA" H 1300 1350 50  0000 C CNN
 F 2 "" H 1300 1500 50  0001 C CNN
@@
 $EndComp
 $Comp
-L GNDA #PWR024
+L GNDA #PWR5
 U 1 1 5A582D37
 P 1300 4700
-F 0 "#PWR024" H 1300 4450 50  0001 C CNN
+F 0 "#PWR5" H 1300 4450 50  0001 C CNN
 F 1 "GNDA" H 1300 4550 50  0000 C CNN
 F 2 "" H 1300 4700 50  0001 C CNN
@@
 $EndComp
 $Comp
-L GNDA #PWR025
+L GNDA #PWR6
 U 1 1 5A582DC6
 P 1350 6250
-F 0 "#PWR025" H 1350 6000 50  0001 C CNN
+F 0 "#PWR6" H 1350 6000 50  0001 C CNN
 F 1 "GNDA" H 1350 6100 50  0000 C CNN
 F 2 "" H 1350 6250 50  0001 C CNN
@@
 $EndComp
 $Comp
-L GNDA #PWR026
+L GNDA #PWR1
 U 1 1 5A583669
 P 1200 6900
-F 0 "#PWR026" H 1200 6650 50  0001 C CNN
+F 0 "#PWR1" H 1200 6650 50  0001 C CNN
 F 1 "GNDA" H 1200 6750 50  0000 C CNN
 F 2 "" H 1200 6900 50  0001 C CNN
@@
 $EndComp
 $Comp
-L GNDA #PWR027
+L GNDA #PWR2
 U 1 1 5A59E351
 P 1200 7550
-F 0 "#PWR027" H 1200 7300 50  0001 C CNN
+F 0 "#PWR2" H 1200 7300 50  0001 C CNN
 F 1 "GNDA" H 1200 7400 50  0000 C CNN
 F 2 "" H 1200 7550 50  0001 C CNN
@@
 $EndComp
 $Comp
-L +3.3V #PWR028
+L +3.3V #PWR34
 U 1 1 5A5B50A6
 P 10400 2300
-F 0 "#PWR028" H 10400 2150 50  0001 C CNN
+F 0 "#PWR34" H 10400 2150 50  0001 C CNN
 F 1 "+3.3V" H 10400 2440 50  0000 C CNN
 F 2 "" H 10400 2300 50  0001 C CNN
@@
 $EndComp
 $Comp
-L GND #PWR029
+L GND #PWR35
 U 1 1 5A5B5168
 P 10400 3250
-F 0 "#PWR029" H 10400 3000 50  0001 C CNN
+F 0 "#PWR35" H 10400 3000 50  0001 C CNN
 F 1 "GND" H 10400 3100 50  0000 C CNN
 F 2 "" H 10400 3250 50  0001 C CNN
@@
 	7900 5650 7900 5300
 Wire Wire Line
-	9700 5050 9850 5050
-Wire Wire Line
-	10150 5050 10750 5050
+	9700 5050 10750 5050
 Wire Wire Line
 	10300 5050 10300 5150
@@
 	4550 6800 4550 6700
 $Comp
-L +3.3V #PWR030
+L +3.3V #PWR15
 U 1 1 5A51A868
 P 3700 3100
-F 0 "#PWR030" H 3700 2950 50  0001 C CNN
+F 0 "#PWR15" H 3700 2950 50  0001 C CNN
 F 1 "+3.3V" H 3700 3240 50  0000 C CNN
 F 2 "" H 3700 3100 50  0001 C CNN
@@
 $EndComp
 $Comp
-L VCC #PWR031
+L VCC #PWR25
 U 1 1 5A51CA39
 P 7600 4550
-F 0 "#PWR031" H 7600 4400 50  0001 C CNN
+F 0 "#PWR25" H 7600 4400 50  0001 C CNN
 F 1 "VCC" H 7600 4700 50  0000 C CNN
 F 2 "" H 7600 4550 50  0001 C CNN
@@
 $EndComp
 $Comp
-L VCC #PWR032
+L VCC #PWR22
 U 1 1 5A51CAA5
 P 6500 3800
-F 0 "#PWR032" H 6500 3650 50  0001 C CNN
+F 0 "#PWR22" H 6500 3650 50  0001 C CNN
 F 1 "VCC" H 6500 3950 50  0000 C CNN
 F 2 "" H 6500 3800 50  0001 C CNN
@@
 $EndComp
 $Comp
-L VCC #PWR033
+L VCC #PWR24
 U 1 1 5A51D5B9
 P 7250 2100
-F 0 "#PWR033" H 7250 1950 50  0001 C CNN
+F 0 "#PWR24" H 7250 1950 50  0001 C CNN
 F 1 "VCC" H 7250 2250 50  0000 C CNN
 F 2 "" H 7250 2100 50  0001 C CNN
@@
 Connection ~ 4800 1800
 $Comp
-L GND #PWR034
+L GND #PWR17
 U 1 1 5A823726
 P 4100 1800
-F 0 "#PWR034" H 4100 1550 50  0001 C CNN
+F 0 "#PWR17" H 4100 1550 50  0001 C CNN
 F 1 "GND" H 4100 1650 50  0000 C CNN
 F 2 "" H 4100 1800 50  0001 C CNN
@@
 Wire Wire Line
 	4800 1100 4800 1200
+$Comp
+L C C6
+U 1 1 5B1494F2
+P 7600 5000
+F 0 "C6" H 7625 5100 50  0000 L CNN
+F 1 "4.7u" H 7625 4900 50  0000 L CNN
+F 2 "" H 7638 4850 50  0001 C CNN
+F 3 "" H 7600 5000 50  0001 C CNN
+	1    7600 5000
+	1    0    0    -1
+$EndComp
+$Comp
+L GND #PWR26
+U 1 1 5B14A011
+P 7600 5250
+F 0 "#PWR26" H 7600 5000 50  0001 C CNN
+F 1 "GND" H 7600 5100 50  0000 C CNN
+F 2 "" H 7600 5250 50  0001 C CNN
+F 3 "" H 7600 5250 50  0001 C CNN
+	1    7600 5250
+	1    0    0    -1
+$EndComp
+Wire Wire Line
+	7600 5250 7600 5150
 $EndSCHEMATC
