File: ADAPTADORESP/WiFiadapter.sch (KiCad schematic (older format))
At the start: 9 parts, among them J1 ADAP_ESP, U1 ESP8266-12E/ESP-12E

Commit message: Adapter_TXRX
TX RX change
Connections:
- net RX: now also J1.9 (Pin_9); no longer J1.7 (Pin_7)
- net TX: now also J1.7 (Pin_7); no longer J1.9 (Pin_9)
Changed lines of the file:
@@
 Text Label 5600 3600 0    60   ~ 0
 SDA
+Text Label 5350 4900 0    60   ~ 0
+TX
 Text Label 5500 4900 0    60   ~ 0
-TX
-Text Label 5350 4900 0    60   ~ 0
 RX
 $Comp

Commit message: Change GPIO16 to GPIO09
Connections:
- net D0: now also U1.11 (IO9); no longer U1.4 (IO16)
Changed lines of the file:
@@
 LIBS:contrib
 LIBS:valves
-LIBS:ESP8266-12E_ESP-12E
 LIBS:WiFiadapter-cache
 EELAYER 25 0
@@
 Text Label 6200 2000 0    60   ~ 0
 TX
-Text Label 6300 2800 0    60   ~ 0
+Text Label 4600 2900 0    60   ~ 0
 D0
 Text Label 4250 1700 0    60   ~ 0
@@
 $EndComp
 NoConn ~ 4750 2300
-NoConn ~ 4750 2900
 NoConn ~ 4750 3000
 $Comp
@@
 	4750 1900 4500 1900
 Wire Wire Line
-	6300 2800 6150 2800
-Wire Wire Line
 	6150 2600 6300 2600
 Wire Wire Line
@@
 Wire Wire Line
 	5700 4500 5700 4900
+Wire Wire Line
+	4750 2900 4600 2900
+NoConn ~ 6150 2800
 $EndSCHEMATC
